File: Continuity Tester.kicad_pcb (KiCad board)
At the start: 2 copper layers, 47.5 x 43 mm, 17 parts, among them J1 Test Probes, SW1 SW_SPST, U1 CA3240

Commit message: Added in the mounting holes
Parts:
- added MH1: MountingHole, MountingHole:MountingHole_3mm, F.Cu at (163.8, 91.4)
- added MH2: MountingHole, MountingHole:MountingHole_3mm, F.Cu at (163.8, 123.2)
- moved R4 18.1 mm to (149.5, 109.5)
- moved BT1 8.43 mm to (156.2, 125.7), turned to 180 degrees
- moved C1 3.81 mm to (159.2, 92.1)
- moved R6 3.81 mm to (149.1, 92.2)
- moved R7 3.81 mm to (151.6, 92.2)
- moved R8 3.81 mm to (156.7, 92.2)
- moved R9 3.81 mm to (154.2, 92.2)
- moved R2 1.42 mm to (141.1, 109.5)
- moved R3 1.42 mm to (145.4, 109.5)
- moved R5 1.42 mm to (137.0, 109.5)
Routing:
- net VCC: track 124.1 -> 82.9 mm
- net GND: track 35.1 -> 0.00 mm
- net Net-(R3-Pad2): track 33.2 -> 13.7 mm
- net +9V: track 24.1 -> 14.4 mm
- net Net-(D1-Pad1): track 97.1 -> 90.6 mm
- net Net-(C1-Pad1): track 21.6 -> 17.6 mm
- net Net-(R7-Pad1): track 27.3 -> 23.4 mm
- net Net-(R5-Pad1): track 35.4 -> 34.6 mm
- added copper zone on B.Cu, net GND
